File: Fuente de tensión regulable/Fuente de tensión regulable.kicad_pcb (KiCad board)
At the start: 2 copper layers, 90 x 58 mm, 35 parts, among them J2 conector DC, J3 conector current, SW1 SW_Wuerth_450301014042, U1 L7805, U3 LM2596S-12

Commit message: Add files via upload
Parts:
- moved D6 0.79 mm to (210.5, 81.5)
Routing:
- net /+: track 162.0 -> 144.1 mm

Commit message: Add files via upload
Parts:
- C2: value 2200uf -> 4900uf
- D4: footprint Diode_SMD:D_SMA -> Diode_THT:D_DO-201AE_P5.08mm_Vertical_AnodeUp
- moved D4 1.20 mm to (164.0, 100.5)
- moved H1 1.00 mm to (176.0, 104.5)
- moved H2 1.00 mm to (186.5, 104.5)
Routing:
- net /Vout+: track 115.2 -> 118.5 mm
- net /Vout-: track 77.7 -> 79.7 mm
Other:
- board text added: "AMP"
- board text added: "ON/OFF"
- board text added: "V"
- board text added: "VOLT"
