File: Fuente de tensión regulable/Fuente de tensión regulable.kicad_sch (KiCad schematic)
At the start: 35 parts, among them J2 conector DC, J3 conector current, SW1 SW_Wuerth_450301014042, U1 L7805, U3 LM2596S-12

Commit message: Add files via upload
Parts:
- C2: value 2200uf -> 4900uf
- D4: footprint Diode_SMD:D_SMA -> Diode_THT:D_DO-201AE_P5.08mm_Vertical_AnodeUp
Other:
- moved on the sheet: C1, C2, D6, H5, H6, SW1
