File: PCB/Fuente de tensión regulable.kicad_pcb (KiCad board)
At the start: 2 copper layers, 90 x 58 mm, 35 parts, among them J2 conector DC, J3 conector current, SW1 SW_Wuerth_450301014042, U1 L7805, U3 LM2596S-12

Commit message: Add files via upload
Parts:
- C7: value 0.1u -> 0.1uf
- D4: renamed from D12; value M4 -> 1N5408
- D5: renamed from D4; value 1N4007 -> 1N5408
- moved C3 0.50 mm to (183.8, 85.5)
- renumbered R34 to POT1, R31 to POT2, R38 to POT3, R32 to R1, R36 to R2, R35 to R3, R37 to R4, R33 to R5
Changed lines of the file:
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@@
 	(net 13 "Net-(SW1-A)")
 	(net 14 "Net-(SS54A-K)")
-	(net 15 "Net-(R34-Pad1)")
+	(net 15 "Net-(POT1-Pad1)")
 	(net 16 "unconnected-(SW1-C-Pad2)")
 	(net 17 "/Vout+")
@@
 		(descr "Diode, DO-201AE series, Axial, Vertical, pin pitch=5.08mm, , length*diameter=9*5.3mm^2, , http://www.farnell.com/datasheets/529758.pdf")
 		(tags "Diode DO-201AE series Axial Vertical pin pitch 5.08mm  length 9mm diameter 5.3mm")
-		(property "Reference" "D4"
+		(property "Reference" "D5"
 			(at 2.54 -3.77 270)
 			(layer "F.SilkS")
@@
 			)
 		)
-		(property "Value" "1N4007"
+		(property "Value" "1N5408"
 			(at 2.54 3.77 270)
 			(layer "F.Fab")
@@
 		(descr "Resistor, Axial_DIN0414 series, Axial, Horizontal, pin pitch=15.24mm, 2W, length*diameter=11.9*4.5mm^2, http://www.vishay.com/docs/20128/wkxwrx.pdf")
 		(tags "Resistor Axial_DIN0414 series Axial Horizontal pin pitch 15.24mm 2W length 11.9mm diameter 4.5mm")
-		(property "Reference" "R33"
+		(property "Reference" "R5"
 			(at 7.62 -3.37 90)
 			(layer "F.SilkS")
@@
 	(footprint "Capacitor_SMD:C_0805_2012Metric_Pad1.18x1.45mm_HandSolder"
 		(layer "F.Cu")
-		(at 183.7875 85)
+		(at 183.8 85.5)
 		(descr "Capacitor SMD 0805 (2012 Metric), square (rectangular) end terminal, IPC_7351 nominal with elongated pad for handsoldering. (Body size source: IPC-SM-782 page 76, https://www.pcb-3d.com/wordpress/wp-content/uploads/ipc-sm-782a_amendment_1_and_2.pdf, https://docs.google.com/spreadsheets/d/1BsfQQcO9C6DZCsRaXUlFlo91Tg2WpOkGARC1WS5S8t0/edit?usp=sharing), generated with kicad-footprint-generator")
 		(tags "capacitor handsolder")
@@
 			)
 		)
-		(property "Description" "Polarized capacitor"
+		(property "Description" "Unpolarized capacitor"
 			(at 0 0 0)
 			(unlocked yes)
@@
 			)
 		)
-		(property ki_fp_filters "CP_*")
+		(property ki_fp_filters "C_*")
 		(sheetname "/")
 		(sheetfile "Fuente de tensión regulable.kicad_sch")
@@
 		(descr "Through hole straight pin header, 1x03, 2.54mm pitch, single row")
 		(tags "Through hole pin header THT 1x03 2.54mm single row")
-		(property "Reference" "R31"
+		(property "Reference" "POT2"
 			(at 0 -2.33 0)
 			(layer "F.SilkS")
@@
 		(descr "Through hole straight pin header, 1x03, 2.54mm pitch, single row")
 		(tags "Through hole pin header THT 1x03 2.54mm single row")
-		(property "Reference" "R38"
+		(property "Reference" "POT3"
 			(at 0 -2.33 0)
 			(layer "F.SilkS")
@@
 		(descr "Resistor SMD 0805 (2012 Metric), square (rectangular) end terminal, IPC_7351 nominal with elongated pad for handsoldering. (Body size source: IPC-SM-782 page 72, https://www.pcb-3d.com/wordpress/wp-content/uploads/ipc-sm-782a_amendment_1_and_2.pdf), generated with kicad-footprint-generator")
 		(tags "resistor handsolder")
-		(property "Reference" "R32"
+		(property "Reference" "R1"
 			(at 0 -1.65 270)
 			(layer "F.SilkS")
@@
 		(descr "Diode, DO-201AE series, Axial, Vertical, pin pitch=5.08mm, , length*diameter=9*5.3mm^2, , http://www.farnell.com/datasheets/529758.pdf")
 		(tags "Diode DO-201AE series Axial Vertical pin pitch 5.08mm  length 9mm diameter 5.3mm")
-		(property "Reference" "D12"
+		(property "Reference" "D4"
 			(at 2.54 -3.77 0)
 			(layer "F.SilkS")
@@
 			)
 		)
-		(property "Value" "M4"
+		(property "Value" "1N5408"
 			(at 2.54 3.77 0)
 			(layer "F.Fab")
@@
 		(descr "Through hole straight pin header, 1x03, 2.54mm pitch, single row")
 		(tags "Through hole pin header THT 1x03 2.54mm single row")
-		(property "Reference" "R34"
+		(property "Reference" "POT1"
 			(at 0 -2.33 0)
 			(layer "F.SilkS")
@@
 			(layers "*.Cu" "*.Mask")
 			(remove_unused_layers no)
-			(net 15 "Net-(R34-Pad1)")
+			(net 15 "Net-(POT1-Pad1)")
 			(pinfunction "1")
 			(pintype "passive")
@@
 		(descr "Resistor SMD 0805 (2012 Metric), square (rectangular) end terminal, IPC_7351 nominal with elongated pad for handsoldering. (Body size source: IPC-SM-782 page 72, https://www.pcb-3d.com/wordpress/wp-content/uploads/ipc-sm-782a_amendment_1_and_2.pdf), generated with kicad-footprint-generator")
 		(tags "resistor handsolder")
-		(property "Reference" "R35"
+		(property "Reference" "R3"
 			(at 0 1.65 90)
 			(layer "B.SilkS")
@@
 			(layers "B.Cu" "B.Mask" "B.Paste")
 			(roundrect_rratio 0.208333)
-			(net 15 "Net-(R34-Pad1)")
+			(net 15 "Net-(POT1-Pad1)")
 			(pintype "passive")
 		)
@@
 		(descr "Resistor SMD 0805 (2012 Metric), square (rectangular) end terminal, IPC_7351 nominal with elongated pad for handsoldering. (Body size source: IPC-SM-782 page 72, https://www.pcb-3d.com/wordpress/wp-content/uploads/ipc-sm-782a_amendment_1_and_2.pdf), generated with kicad-footprint-generator")
 		(tags "resistor handsolder")
-		(property "Reference" "R37"
+		(property "Reference" "R4"
 			(at 0 1.65 90)
 			(layer "B.SilkS")
@@
 			)
 		)
-		(property "Value" "0.1u"
+		(property "Value" "0.1uf"
 			(at 0 -1.68 0)
 			(layer "B.Fab")
@@
 		(descr "Resistor SMD 0805 (2012 Metric), square (rectangular) end terminal, IPC_7351 nominal with elongated pad for handsoldering. (Body size source: IPC-SM-782 page 72, https://www.pcb-3d.com/wordpress/wp-content/uploads/ipc-sm-782a_amendment_1_and_2.pdf), generated with kicad-footprint-generator")
 		(tags "resistor handsolder")
-		(property "Reference" "R36"
+		(property "Reference" "R2"
 			(at 0 1.65 90)
 			(layer "B.SilkS")
@@
 	)
 	(segment
+		(start 182.7625 85.5)
+		(end 182.7625 89.2365)
+		(width 1.5)
+		(layer "F.Cu")
+		(net 8)
+	)
+	(segment
 		(start 163.65 74.45)
 		(end 169.1 74.45)
@@
 	)
 	(segment
+		(start 182.7625 89.2365)
+		(end 182.75 89.249)
+		(width 1.5)
+		(layer "F.Cu")
+		(net 8)
+	)
+	(segment
 		(start 188.5 71.75)
 		(end 186 71.75)
@@
 	)
 	(segment
-		(start 196.078916 68)
-		(end 192.25 68)
-		(width 2.5)
+		(start 182.7625 84.3)
+		(end 182.7625 85.5)
+		(width 1.5)
 		(layer "F.Cu")
 		(net 8)
 	)
 	(segment
-		(start 182.75 84.2875)
-		(end 182.75 89.35)
-		(width 1.5)
+		(start 196.078916 68)
+		(end 192.25 68)
+		(width 2.5)
 		(layer "F.Cu")
 		(net 8)
@@
 		(layer "F.Cu")
 		(net 8)
+	)
+	(segment
+		(start 182.75 84.2875)
+		(end 182.7625 84.3)
+		(width 1.5)
+		(layer "F.Cu")
+		(net 8)
