File: PCB/Fuente de tensión regulable.kicad_sch (KiCad schematic)
At the start: 35 parts, among them J2 conector DC, J3 conector current, SW1 SW_Wuerth_450301014042, U1 L7805, U3 LM2596S-12

Commit message: Add files via upload
Parts:
- removed C3: 1uf, Capacitor_SMD:C_0805_2012Metric_Pad1.18x1.45mm_HandSolder, symbol Device:C_Polarized
- added C3: 1uf, Capacitor_SMD:C_0805_2012Metric_Pad1.18x1.45mm_HandSolder, symbol Device:C
- C7: value 0.1u -> 0.1uf
- D4: renamed from D12; value M4 -> 1N5408
- D5: renamed from D4; value 1N4007 -> 1N5408
- renumbered R34 to POT1, R31 to POT2, R38 to POT3, R32 to R1, R36 to R2, R35 to R3, R37 to R4, R33 to R5
Connections:
- net +: now also C3.1
- net GND: now also C3.2
Other:
- note added: "ALIMENTACIÓN"
- note added: "ALIMENTACIÓN 2"
- note added: "MODULO VOLT-AMPER"
- note added: "PRIMERA ETAPA: REDUCCIÓN Y CONVERSIÓN"
- note added: "SEGUNDA Y TERCERA ETAPA: REGULACIÓN Y SALIDA DE VOLTAJE"
- note added: "led que indica el funcionamiento"
- note removed: "led indicativo que indica el funcionamiento"
- moved on the sheet: A8A, A8B, A8C, C1, C2, C4, C5, C6, C7, D1, D2, D3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
